File: badgelife101/badgelife101.kicad_sch (KiCad schematic)
At the start: 14 parts

Commit message: jlcpcba
Parts:
- BT1: LCSC (none) -> C964831; MFR (none) -> MY-2032-08
- D1, D2, D3, D4, D5, D6: LCSC (none) -> C2286; MFR (none) -> KT-0603R
- R1, R2, R3, R4, R5, R6: value 330 -> 470; LCSC (none) -> C23179; MFR (none) -> 0603WAF4700T5E
Changed lines of the file:
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@@
+      (effects (font (size 1.27 1.27)) hide)
+    )
+    (property "LCSC" "C2286" (at 143.51 87.63 0)
+      (effects (font (size 1.27 1.27)) hide)
+    )
+    (property "MFR" "KT-0603R" (at 143.51 87.63 0)
       (effects (font (size 1.27 1.27)) hide)
     )
@@
       (effects (font (size 1.27 1.27)) (justify left))
     )
-    (property "Value" "330" (at 146.05 81.28 0)
+    (property "Value" "470" (at 146.05 81.28 0)
       (effects (font (size 1.27 1.27)) (justify left))
     )
@@
       (effects (font (size 1.27 1.27)) hide)
     )
+    (property "LCSC" "C23179" (at 143.51 80.01 0)
+      (effects (font (size 1.27 1.27)) hide)
+    )
+    (property "MFR" "0603WAF4700T5E" (at 143.51 80.01 0)
+      (effects (font (size 1.27 1.27)) hide)
+    )
     (pin "1")
     (pin "2")
@@
       (effects (font (size 1.27 1.27)) hide)
     )
+    (property "LCSC" "" (at 91.44 92.71 0)
+      (effects (font (size 1.27 1.27)) hide)
+    )
+    (property "MFR" "" (at 91.44 92.71 0)
+      (effects (font (size 1.27 1.27)) hide)
+    )
     (pin "1")
     (instances
@@
       (effects (font (size 1.27 1.27)) hide)
     )
+    (property "LCSC" "C964831" (at 91.44 88.9 0)
+      (effects (font (size 1.27 1.27)) hide)
+    )
+    (property "MFR" "MY-2032-08" (at 91.44 88.9 0)
+      (effects (font (size 1.27 1.27)) hide)
+    )
     (pin "1")
     (pin "2")
@@
       (effects (font (size 1.27 1.27)) (justify left))
     )
-    (property "Value" "330" (at 163.83 81.28 0)
+    (property "Value" "470" (at 163.83 81.28 0)
       (effects (font (size 1.27 1.27)) (justify left))
     )
@@
       (effects (font (size 1.27 1.27)) hide)
     )
+    (property "LCSC" "C23179" (at 161.29 80.01 0)
+      (effects (font (size 1.27 1.27)) hide)
+    )
+    (property "MFR" "0603WAF4700T5E" (at 161.29 80.01 0)
+      (effects (font (size 1.27 1.27)) hide)
+    )
     (pin "1")
     (pin "2")
@@
       (effects (font (size 1.27 1.27)) hide)
     )
+    (property "LCSC" "C2286" (at 170.18 87.63 0)
+      (effects (font (size 1.27 1.27)) hide)
+    )
+    (property "MFR" "KT-0603R" (at 170.18 87.63 0)
+      (effects (font (size 1.27 1.27)) hide)
+    )
     (pin "1")
     (pin "2")
@@
       (effects (font (size 1.27 1.27)) hide)
     )
+    (property "LCSC" "C2286" (at 125.73 87.63 0)
+      (effects (font (size 1.27 1.27)) hide)
+    )
+    (property "MFR" "KT-0603R" (at 125.73 87.63 0)
+      (effects (font (size 1.27 1.27)) hide)
+    )
     (pin "1")
     (pin "2")
@@
       (effects (font (size 1.27 1.27)) hide)
     )
+    (property "LCSC" "C2286" (at 134.62 87.63 0)
+      (effects (font (size 1.27 1.27)) hide)
+    )
+    (property "MFR" "KT-0603R" (at 134.62 87.63 0)
+      (effects (font (size 1.27 1.27)) hide)
+    )
     (pin "1")
     (pin "2")
@@
       (effects (font (size 1.27 1.27)) (justify left))
     )
-    (property "Value" "330" (at 128.27 81.28 0)
+    (property "Value" "470" (at 128.27 81.28 0)
       (effects (font (size 1.27 1.27)) (justify left))
     )
@@
       (effects (font (size 1.27 1.27)) hide)
     )
+    (property "LCSC" "C23179" (at 125.73 80.01 0)
+      (effects (font (size 1.27 1.27)) hide)
+    )
+    (property "MFR" "0603WAF4700T5E" (at 125.73 80.01 0)
+      (effects (font (size 1.27 1.27)) hide)
+    )
     (pin "1")
     (pin "2")
@@
       (effects (font (size 1.27 1.27)) hide)
     )
+    (property "LCSC" "C2286" (at 152.4 87.63 0)
+      (effects (font (size 1.27 1.27)) hide)
+    )
+    (property "MFR" "KT-0603R" (at 152.4 87.63 0)
+      (effects (font (size 1.27 1.27)) hide)
+    )
     (pin "1")
     (pin "2")
@@
       (effects (font (size 1.27 1.27)) (justify left))
     )
-    (property "Value" "330" (at 172.72 81.28 0)
+    (property "Value" "470" (at 172.72 81.28 0)
       (effects (font (size 1.27 1.27)) (justify left))
     )
@@
       (effects (font (size 1.27 1.27)) hide)
     )
+    (property "LCSC" "C23179" (at 170.18 80.01 0)
+      (effects (font (size 1.27 1.27)) hide)
+    )
+    (property "MFR" "0603WAF4700T5E" (at 170.18 80.01 0)
+      (effects (font (size 1.27 1.27)) hide)
+    )
     (pin "1")
     (pin "2")
@@
       (effects (font (size 1.27 1.27)) hide)
     )
+    (property "LCSC" "C2286" (at 161.29 87.63 0)
+      (effects (font (size 1.27 1.27)) hide)
+    )
+    (property "MFR" "KT-0603R" (at 161.29 87.63 0)
+      (effects (font (size 1.27 1.27)) hide)
+    )
     (pin "1")
     (pin "2")
@@
       (effects (font (size 1.27 1.27)) (justify left))
     )
-    (property "Value" "330" (at 137.16 81.28 0)
+    (property "Value" "470" (at 137.16 81.28 0)
       (effects (font (size 1.27 1.27)) (justify left))
     )
@@
       (effects (font (size 1.27 1.27)) hide)
     )
+    (property "LCSC" "C23179" (at 134.62 80.01 0)
+      (effects (font (size 1.27 1.27)) hide)
+    )
+    (property "MFR" "0603WAF4700T5E" (at 134.62 80.01 0)
+      (effects (font (size 1.27 1.27)) hide)
+    )
     (pin "1")
     (pin "2")
@@
       (effects (font (size 1.27 1.27)) (justify left))
     )
-    (property "Value" "330" (at 154.94 81.28 0)
+    (property "Value" "470" (at 154.94 81.28 0)
       (effects (font (size 1.27 1.27)) (justify left))
     )
@@
       (effects (font (size 1.27 1.27)) hide)
     )
+    (property "LCSC" "C23179" (at 152.4 80.01 0)
+      (effects (font (size 1.27 1.27)) hide)
+    )
+    (property "MFR" "0603WAF4700T5E" (at 152.4 80.01 0)
+      (effects (font (size 1.27 1.27)) hide)
+    )
